Commit message: fix head position of staro for gazebo

File: hrpsys_gazebo_tutorials/robot_models/STARO/STARO_with_hand.urdf.xacro (robot description, xacro)
@@ -6,5 +6,5 @@
     <parent link="HEAD_LINK1" />
     <child  link="head" />
-    <origin xyz="0.075 0 0.15" rpy="0 0 0"/>
+    <origin xyz="0.07595 0 0.19825" rpy="0 0 0"/>
   </joint>
   <xacro:robotiq_hand_for_gazebo prefix="L_" parent="LARM_LINK7">
