Commit message: fix staro model for using multisense

File: hrpsys_ros_bridge_tutorials/models/STARO.urdf.xacro (robot description, xacro)
@@ -1,5 +1,6 @@
 <robot xmlns:xacro="http://www.ros.org/wiki/xacro" name="STARO" >
   <xacro:include filename="STARO_body.urdf" />
-  <xacro:include filename="$(find multisense_sl_description)/urdf/multisense_sl_v4.urdf" />
+  <!-- no head for REAL multisense -->
+  <!--xacro:include filename="$(find multisense_description)/urdf/multisenseSL.urdf" /-->
   <xacro:include filename="$(find robotiq_hand_description)/urdf/robotiq_hand.urdf.xacro" />
   <link name="HEAD_LINK1">
@@ -16,5 +17,5 @@
       </geometry>
     </collision>
-    <inertial>
+    <inertial> <!-- mass propaties should be corrected -->
       <mass value="4.873" />
       <origin xyz="0.01617 0.00844 0.1502" rpy="0 -0 0"/>
@@ -26,7 +27,9 @@
     <mu2>0.9</mu2>
   </gazebo>
+  <link name="multisense/head_root" />
   <joint name="staro_to_multisense" type="fixed">
     <parent link="HEAD_LINK1" />
-    <child  link="head" />
+    <!--child  link="head" /--> <!-- for drcsim / multisense_sl_description -->
+    <child  link="multisense/head_root" /> <!-- for multisense / multisense_description -->
     <origin xyz="0.07595 0 0.19825" rpy="0 0 0"/>
   </joint>
@@ -44,5 +47,5 @@
       </geometry>
     </collision>
-    <inertial>
+    <inertial> <!-- mass propaties should be corrected -->
       <mass value="4.219" />
       <origin xyz="-0.02359 0.12884 -0.02825" rpy="0 -0 0"/>
@@ -67,5 +70,5 @@
       </geometry>
     </collision>
-    <inertial>
+    <inertial> <!-- mass propaties should be corrected -->
       <mass value="4.219" />
       <origin xyz="0.02359 -0.12884 -0.02825" rpy="0 -0 0"/>

Commit message: add xacro file for robotiq hand

File: hrpsys_ros_bridge_tutorials/models/STARO.urdf.xacro (robot description, xacro)
@@ -80,9 +80,5 @@
     <mu2>0.9</mu2>
   </gazebo>
-  <xacro:robotiq_hand prefix="L_" parent="LARM_LINK7" reflect="-1">
-    <origin xyz="-0.027224 0.149 -0.027224" rpy="-1.5707963268 -0.7853981634 3.1415926536" />
-  </xacro:robotiq_hand>
-  <xacro:robotiq_hand prefix="R_" parent="RARM_LINK7" reflect="-1">
-    <origin xyz="-0.027224 -0.149 -0.027224" rpy="-1.5707963268 -0.7853981634 3.1415926536" />
-  </xacro:robotiq_hand>
+  <xacro:include filename="$(find hrpsys_ros_bridge_tutorials)/models/robotiq_l.urdf.xacro" />
+  <xacro:include filename="$(find hrpsys_ros_bridge_tutorials)/models/robotiq_r.urdf.xacro" />
 </robot>

Commit message: update camera offset parameter for staro

File: hrpsys_ros_bridge_tutorials/models/STARO.urdf.xacro (robot description, xacro)
@@ -31,5 +31,6 @@
     <!--child  link="head" /--> <!-- for drcsim / multisense_sl_description -->
     <child  link="multisense/head_root" /> <!-- for multisense / multisense_description -->
-    <origin xyz="0.07595 0 0.19825" rpy="0 0 0"/>
+    <!--origin xyz="0.07595 0 0.19825" rpy="0 0 0"/-->
+    <origin xyz="0.0832703049 -0.0076383991 0.1989256909" rpy="0.0288834088 0.0091750864 0.0131467637" /> <!-- calibrated 2015.01.21-->
   </joint>
   <link name="LARM_LINK7">
@@ -81,3 +82,11 @@
   <xacro:include filename="$(find hrpsys_ros_bridge_tutorials)/models/robotiq_l.urdf.xacro" />
   <xacro:include filename="$(find hrpsys_ros_bridge_tutorials)/models/robotiq_r.urdf.xacro" />
+  <!-- for calibration / original offset of camera_frame
+  <link name="multisense/left_camera_optical_frame" />
+  <joint name="multisense/left_camera_optical_frame_joint" type="fixed">
+    <parent link="HEAD_LINK1" />
+    <child  link="multisense/left_camera_optical_frame" />
+    <origin xyz="0.07595 0.035 0.19625" rpy="-1.5707960129 0 -1.5707960129"/>
+  </joint>
+  -->
 </robot>
