Commit message: [hrpsys_ros_bridge_tutorials] Update HRP2JSKNT model to be with multisense SL

File: hrpsys_ros_bridge_tutorials/models/HRP2JSKNT.urdf.xacro (robot description, xacro)
@@ -3,3 +3,11 @@
   <xacro:include filename="HRP3HAND_L.urdf" />
   <xacro:include filename="HRP3HAND_R.urdf" />
+  <xacro:include filename="$(find multisense_description)/urdf/multisenseSL.urdf" />
+  <joint name="hrp2_to_multisense" type="fixed">
+    <parent link="HEAD_LINK1" />
+    <!--child  link="head" /--> <!-- for drcsim / multisense_sl_description -->
+    <child  link="head_root" /> <!-- for multisense / multisense_description -->
+    <!--origin xyz="0.07595 0 0.19825" rpy="0 0 0"/-->
+    <origin xyz="0.0 0.0 0.1" rpy="0 0 0" /> <!-- calibrated 2015.01.21-->
+  </joint>
 </robot>
