Commit message: fix jaxon model

File: hrpsys_ros_bridge_tutorials/models/JAXON.urdf.xacro (robot description, xacro)
@@ -36,5 +36,5 @@
       <origin xyz="0 0.0 0" rpy="0 -0 0"/>
       <geometry>
-        <mesh filename="package://hrpsys_ros_bridge_tutorials/models/JAXON_meshes/l_hand_attached_link.dae" scale="0.0254 0.0254 0.0254" />
+        <mesh filename="package://hrpsys_ros_bridge_tutorials/models/JAXON_meshes/l_hand_attached_link.dae" scale="1 1 1" />
       </geometry>
     </visual>
@@ -42,5 +42,5 @@
       <origin xyz="0 0.0 0" rpy="0 -0 0"/>
       <geometry>
-        <mesh filename="package://hrpsys_ros_bridge_tutorials/models/JAXON_meshes/l_hand_attached_link.dae" scale="0.0254 0.0254 0.0254" />
+        <mesh filename="package://hrpsys_ros_bridge_tutorials/models/JAXON_meshes/l_hand_attached_link.dae" scale="1 1 1" />
       </geometry>
     </collision>
@@ -60,5 +60,5 @@
       <origin xyz="0 0 0" rpy="0 -0 0"/>
       <geometry>
-        <mesh filename="package://hrpsys_ros_bridge_tutorials/models/JAXON_meshes/r_hand_attached_link.dae" scale="0.0254 0.0254 0.0254" />
+        <mesh filename="package://hrpsys_ros_bridge_tutorials/models/JAXON_meshes/r_hand_attached_link.dae" scale="1 1 1" />
       </geometry>
     </visual>
@@ -66,5 +66,5 @@
       <origin xyz="0 0 0" rpy="0 -0 0"/>
       <geometry>
-        <mesh filename="package://hrpsys_ros_bridge_tutorials/models/JAXON_meshes/r_hand_attached_link.dae" scale="0.0254 0.0254 0.0254" />
+        <mesh filename="package://hrpsys_ros_bridge_tutorials/models/JAXON_meshes/r_hand_attached_link.dae" scale="1 1 1" />
       </geometry>
     </collision>

Commit message: update generation method for JAXON urdf

File: hrpsys_ros_bridge_tutorials/models/JAXON.urdf.xacro (robot description, xacro)
@@ -1,34 +1,4 @@
 <robot xmlns:xacro="http://www.ros.org/wiki/xacro" name="JAXON" >
   <xacro:include filename="JAXON_body.urdf" />
-  <link name="HEAD_LINK1">
-    <visual>
-      <origin xyz="0 0 0" rpy="0 -0 0"/>
-      <geometry>
-        <mesh filename="package://hrpsys_ros_bridge_tutorials/models/JAXON_meshes/HEAD_LINK1_without_camera.dae" scale="1 1 1" />
-      </geometry>
-    </visual>
-    <collision>
-      <origin xyz="0 0 0" rpy="0 -0 0"/>
-      <geometry>
-        <mesh filename="package://hrpsys_ros_bridge_tutorials/models/JAXON_meshes/HEAD_LINK1_without_camera.dae" scale="1 1 1" />
-      </geometry>
-    </collision>
-    <inertial> <!-- mass propaties should be corrected -->
-      <mass value="4.873" />
-      <origin xyz="0.01617 0.00844 0.1502" rpy="0 -0 0"/>
-      <inertia ixx="0.15" ixy="1.76326e-18" ixz="0.01" iyy="0.16" iyz="-1.33463e-17" izz="0.04"/>
-    </inertial>
-  </link>
-  <gazebo reference="HEAD_LINK1">
-    <mu1>0.9</mu1>
-    <mu2>0.9</mu2>
-  </gazebo>
-  <link name="multisense/head_root" />
-  <joint name="head_tip_to_multisense" type="fixed">
-    <parent link="HEAD_LINK1" />
-    <!--child  link="head" /--> <!-- for drcsim / multisense_sl_description -->
-    <child  link="multisense/head_root" /> <!-- for multisense / multisense_description -->
-    <origin xyz="0.1005 0 0.05625" rpy="0 0 0"/>
-  </joint>
   <!-- -->
   <link name="LARM_LINK7">
@@ -79,19 +49,18 @@
     <mu2>0.9</mu2>
   </gazebo>
+  <!-- HEAD -->
+  <xacro:include filename="$(find multisense_description)/urdf/multisenseSL.urdf" />
+  <joint name="head_tip_to_multisense" type="fixed">
+    <parent link="HEAD_LINK1" />
+    <child  link="head_root" />
+    <origin xyz="0.1005 0 0.05625" rpy="0 0 0"/>
+  </joint>
   <!-- HAND -->
   <xacro:include filename="$(find jaxon_description)/urdf/thk_hand.urdf.xacro" />
   <xacro:thk_hand prefix="L_" parent="LARM_LINK7" type="revolute">
-    <origin xyz="0 0 -0.095" rpy="-1.5707963268 1.5707963268 0" />
+    <origin xyz="0 0 -0.085" rpy="0 1.5707963268 0" />
   </xacro:thk_hand>
   <xacro:thk_hand prefix="R_" parent="RARM_LINK7" type="revolute">
-    <origin xyz="0 0 -0.095" rpy="1.5707963268 1.5707963268 0" />
+    <origin xyz="0 0 -0.085" rpy="0 1.5707963268 0" />
   </xacro:thk_hand>
-  <!-- for calibration / original offset of camera_frame
-  <link name="multisense/left_camera_optical_frame" />
-  <joint name="multisense/left_camera_optical_frame_joint" type="fixed">
-    <parent link="HEAD_LINK1" />
-    <child  link="multisense/left_camera_optical_frame" />
-    <origin xyz="0.07595 0.035 0.19625" rpy="-1.5707960129 0 -1.5707960129"/>
-  </joint>
-  -->
 </robot>

Commit message: [hrpsys_ros_bridge_tutorials] Update jaxon calibration parameter

File: hrpsys_ros_bridge_tutorials/models/JAXON.urdf.xacro (robot description, xacro)
@@ -54,5 +54,5 @@
     <parent link="HEAD_LINK1" />
     <child  link="head_root" />
-    <origin xyz="0.1005 0 0.05625" rpy="0 0 0"/>
+    <origin rpy="0.004 0.01 0.01" xyz="0.1005 0 0.07625"/>
   </joint>
   <!-- HAND -->

Commit message: update jaxon hand type from 002 to 003

File: hrpsys_ros_bridge_tutorials/models/JAXON.urdf.xacro (robot description, xacro)
@@ -57,10 +57,10 @@
   </joint>
   <!-- HAND -->
-  <xacro:include filename="$(find jaxon_description)/urdf/thk_hand002.urdf.xacro" />
+  <xacro:include filename="$(find jaxon_description)/urdf/thk_hand003.urdf.xacro" />
   <xacro:thk_hand prefix="L_" parent="LARM_LINK7" type="revolute">
-    <origin xyz="0 0 -0.085" rpy="0 1.5707963268 0" />
+    <origin xyz="0 0 -0.085" rpy="-1.5707963268 1.5707963268 0" />
   </xacro:thk_hand>
   <xacro:thk_hand prefix="R_" parent="RARM_LINK7" type="revolute">
-    <origin xyz="0 0 -0.085" rpy="0 1.5707963268 0" />
+    <origin xyz="0 0 -0.085" rpy="1.5707963268 1.5707963268 0" />
   </xacro:thk_hand>
 </robot>

Commit message: [hrpsys_ros_bridge_tutorails] Update hand/eye/leg calib parameter for JAXON by hand

File: hrpsys_ros_bridge_tutorials/models/JAXON.urdf.xacro (robot description, xacro)
@@ -54,5 +54,7 @@
     <parent link="HEAD_LINK1" />
     <child  link="head_root" />
-    <origin rpy="0.004 0.01 0.01" xyz="0.1005 0 0.07625"/>
+    <!-- <origin rpy="-0.01 0.01 0.017" xyz="0.08 0.01 0.045"/> --> <!-- For leg -->
+    <origin rpy="-0.01 0.01 0.017" xyz="0.09 0.01 0.055"/> <!--middle-->
+    <!-- <origin rpy="-0.01 0.01 0.017" xyz="0.10 0.01 0.065"/> --> <!-- For hand -->
   </joint>
   <!-- HAND -->

Commit message: [hrpsys_ros_bridge_tutorials] update jaxon urdf

File: hrpsys_ros_bridge_tutorials/models/JAXON.urdf.xacro (robot description, xacro)
@@ -55,5 +55,6 @@
     <child  link="head_root" />
     <!-- <origin rpy="-0.01 0.01 0.017" xyz="0.08 0.01 0.045"/> --> <!-- For leg -->
-    <origin rpy="-0.01 0.01 0.017" xyz="0.09 0.01 0.055"/> <!--middle-->
+    <origin rpy="-0.01 0.02 0.017" xyz="0.07 -0.01 0.045"/>
+    <!-- <origin rpy="-0.01 0.01 0.017" xyz="0.09 0.01 0.055"/>  --><!--middle-->
     <!-- <origin rpy="-0.01 0.01 0.017" xyz="0.10 0.01 0.065"/> --> <!-- For hand -->
   </joint>

Commit message: [hrpsys_ros_bridge_tutorials] Update jaxon's leg/eye calib param

File: hrpsys_ros_bridge_tutorials/models/JAXON.urdf.xacro (robot description, xacro)
@@ -55,5 +55,6 @@
     <child  link="head_root" />
     <!-- <origin rpy="-0.01 0.01 0.017" xyz="0.08 0.01 0.045"/> --> <!-- For leg -->
-    <origin rpy="-0.01 0.02 0.017" xyz="0.07 -0.01 0.045"/>
+    <origin rpy="-0.01 0.035 -0.005" xyz="0.085 0.01 0.065"/>
+    <!-- <rigin rpy="-0.01 0.02 0.017" xyz="0.07 -0.01 0.045"/> old -->
     <!-- <origin rpy="-0.01 0.01 0.017" xyz="0.09 0.01 0.055"/>  --><!--middle-->
     <!-- <origin rpy="-0.01 0.01 0.017" xyz="0.10 0.01 0.065"/> --> <!-- For hand -->

Commit message: [hrpsys_ros_bridge_tutorials] Use jsk_model's hand attachmend collada file in JAXON models

File: hrpsys_ros_bridge_tutorials/models/JAXON.urdf.xacro (robot description, xacro)
@@ -6,5 +6,5 @@
       <origin xyz="0 0.0 0" rpy="0 -0 0"/>
       <geometry>
-        <mesh filename="package://hrpsys_ros_bridge_tutorials/models/JAXON_meshes/l_hand_attached_link.dae" scale="1 1 1" />
+        <mesh filename="package://jsk_models/JAXON/l_hand_attached_link.dae" scale="1 1 1" />
       </geometry>
     </visual>
@@ -12,5 +12,5 @@
       <origin xyz="0 0.0 0" rpy="0 -0 0"/>
       <geometry>
-        <mesh filename="package://hrpsys_ros_bridge_tutorials/models/JAXON_meshes/l_hand_attached_link.dae" scale="1 1 1" />
+        <mesh filename="package://jsk_models/JAXON/l_hand_attached_link.dae" scale="1 1 1" />
       </geometry>
     </collision>
@@ -30,5 +30,5 @@
       <origin xyz="0 0 0" rpy="0 -0 0"/>
       <geometry>
-        <mesh filename="package://hrpsys_ros_bridge_tutorials/models/JAXON_meshes/r_hand_attached_link.dae" scale="1 1 1" />
+        <mesh filename="package://jsk_models/JAXON/r_hand_attached_link.dae" scale="1 1 1" />
       </geometry>
     </visual>
@@ -36,5 +36,5 @@
       <origin xyz="0 0 0" rpy="0 -0 0"/>
       <geometry>
-        <mesh filename="package://hrpsys_ros_bridge_tutorials/models/JAXON_meshes/r_hand_attached_link.dae" scale="1 1 1" />
+        <mesh filename="package://jsk_models/JAXON/r_hand_attached_link.dae" scale="1 1 1" />
       </geometry>
     </collision>

File: hrpsys_ros_bridge_tutorials/models/JAXON_RED.urdf.xacro (robot description, xacro)
@@ -6,5 +6,5 @@
       <origin xyz="0 0.0 0" rpy="0 -0 0"/>
       <geometry>
-        <mesh filename="package://hrpsys_ros_bridge_tutorials/models/JAXON_RED_meshes/l_hand_attached_link.dae" scale="1 1 1" />
+        <mesh filename="package://jsk_models/JAXON/l_hand_attached_link.dae" scale="1 1 1" />
       </geometry>
     </visual>
@@ -12,5 +12,5 @@
       <origin xyz="0 0.0 0" rpy="0 -0 0"/>
       <geometry>
-        <mesh filename="package://hrpsys_ros_bridge_tutorials/models/JAXON_RED_meshes/l_hand_attached_link.dae" scale="1 1 1" />
+        <mesh filename="package://jsk_models/JAXON/l_hand_attached_link.dae" scale="1 1 1" />
       </geometry>
     </collision>
@@ -30,5 +30,5 @@
       <origin xyz="0 0 0" rpy="0 -0 0"/>
       <geometry>
-        <mesh filename="package://hrpsys_ros_bridge_tutorials/models/JAXON_RED_meshes/r_hand_attached_link.dae" scale="1 1 1" />
+        <mesh filename="package://jsk_models/JAXON/r_hand_attached_link.dae" scale="1 1 1" />
       </geometry>
     </visual>
@@ -36,5 +36,5 @@
       <origin xyz="0 0 0" rpy="0 -0 0"/>
       <geometry>
-        <mesh filename="package://hrpsys_ros_bridge_tutorials/models/JAXON_RED_meshes/r_hand_attached_link.dae" scale="1 1 1" />
+        <mesh filename="package://jsk_models/JAXON/r_hand_attached_link.dae" scale="1 1 1" />
       </geometry>
     </collision>

Commit message: [hrpsys_ros_bridge_tutorials] Calibrate multisense external parameters of JAXON for new head

File: hrpsys_ros_bridge_tutorials/models/JAXON.urdf.xacro (robot description, xacro)
@@ -55,8 +55,9 @@
     <child  link="head_root" />
     <!-- <origin rpy="-0.01 0.01 0.017" xyz="0.08 0.01 0.045"/> --> <!-- For leg -->
-    <origin rpy="-0.01 0.035 -0.005" xyz="0.085 0.01 0.065"/>
     <!-- <rigin rpy="-0.01 0.02 0.017" xyz="0.07 -0.01 0.045"/> old -->
     <!-- <origin rpy="-0.01 0.01 0.017" xyz="0.09 0.01 0.055"/>  --><!--middle-->
     <!-- <origin rpy="-0.01 0.01 0.017" xyz="0.10 0.01 0.065"/> --> <!-- For hand -->
+    <!-- <origin rpy="-0.01 0.035 -0.005" xyz="0.085 0.01 0.065"/> --> <!-- old head in 20151022 -->
+    <origin rpy="-0.004 0.275 -0.01" xyz="0.1 0.01 0.085"/> <!-- new head in 20151022 -->
   </joint>
   <!-- HAND -->

Commit message: [hrpsys_ros_brige_tutorials] Adjust multisense location in JAXON1

File: hrpsys_ros_bridge_tutorials/models/JAXON.urdf.xacro (robot description, xacro)
@@ -59,5 +59,6 @@
     <!-- <origin rpy="-0.01 0.01 0.017" xyz="0.10 0.01 0.065"/> --> <!-- For hand -->
     <!-- <origin rpy="-0.01 0.035 -0.005" xyz="0.085 0.01 0.065"/> --> <!-- old head in 20151022 -->
-    <origin rpy="-0.004 0.275 -0.01" xyz="0.1 0.01 0.085"/> <!-- new head in 20151022 -->
+    <!-- <origin rpy="-0.004 0.275 -0.01" xyz="0.1 0.01 0.085"/> --> <!-- new head in 20151022 -->
+    <origin rpy="0.003 0.255 -0.02" xyz="0.1 0.01 0.085"/> <!-- new head in 20151125 -->
   </joint>
   <!-- HAND -->

Commit message: [hrpsys_ros_bridge_tutorials] Reflect reverting old head mount for multisense of JAXON1

File: hrpsys_ros_bridge_tutorials/models/JAXON.urdf.xacro (robot description, xacro)
@@ -60,5 +60,6 @@
     <!-- <origin rpy="-0.01 0.035 -0.005" xyz="0.085 0.01 0.065"/> --> <!-- old head in 20151022 -->
     <!-- <origin rpy="-0.004 0.275 -0.01" xyz="0.1 0.01 0.085"/> --> <!-- new head in 20151022 -->
-    <origin rpy="0.003 0.255 -0.02" xyz="0.1 0.01 0.085"/> <!-- new head in 20151125 -->
+    <!-- <origin rpy="0.003 0.255 -0.02" xyz="0.1 0.01 0.085"/> --> <!-- new head in 20151125 -->
+    <origin rpy="0.015 0.035 -0.02" xyz="0.085 0.01 0.085"/> <!-- revert to old head in 20151127 -->
   </joint>
   <!-- HAND -->
