Commit message: [hrpsys_ros_bridge_tutorials] Update calib parameter for jaxon red

File: hrpsys_ros_bridge_tutorials/models/JAXON_RED.urdf.xacro (robot description, xacro)
@@ -55,5 +55,6 @@
     <child  link="head_root" />
     <!-- <origin rpy="-0.01 0.01 0.017" xyz="0.08 0.01 0.045"/> --> <!-- For leg -->
-    <origin rpy="-0.01 0.01 0.017" xyz="0.09 0.01 0.055"/> <!--middle-->
+    <!-- <origin rpy="-0.01 0.04 0.017" xyz="0.095 -0.01 0.055"/> for jaxon -->
+    <origin rpy="-0.01 0.04 -0.01" xyz="0.09 0.01 0.1"/> <!--for jaxon red-->
     <!-- <origin rpy="-0.01 0.01 0.017" xyz="0.10 0.01 0.065"/> --> <!-- For hand -->
   </joint>

Commit message: [hrpsys_ros_bridge_tutorials] Update hand/eye parameter for jaxon red

File: hrpsys_ros_bridge_tutorials/models/JAXON_RED.urdf.xacro (robot description, xacro)
@@ -56,5 +56,5 @@
     <!-- <origin rpy="-0.01 0.01 0.017" xyz="0.08 0.01 0.045"/> --> <!-- For leg -->
     <!-- <origin rpy="-0.01 0.04 0.017" xyz="0.095 -0.01 0.055"/> for jaxon -->
-    <origin rpy="-0.01 0.04 -0.01" xyz="0.09 0.01 0.1"/> <!--for jaxon red-->
+    <origin rpy="-0.01 0.04 -0.01" xyz="0.09 0.01 0.055"/> <!--for jaxon red-->
     <!-- <origin rpy="-0.01 0.01 0.017" xyz="0.10 0.01 0.065"/> --> <!-- For hand -->
   </joint>

Commit message: [hrpsys_ros_bridge_tutorials] Update calib paraemeter for kawada leg

File: hrpsys_ros_bridge_tutorials/models/JAXON_RED.urdf.xacro (robot description, xacro)
@@ -56,5 +56,6 @@
     <!-- <origin rpy="-0.01 0.01 0.017" xyz="0.08 0.01 0.045"/> --> <!-- For leg -->
     <!-- <origin rpy="-0.01 0.04 0.017" xyz="0.095 -0.01 0.055"/> for jaxon -->
-    <origin rpy="-0.01 0.04 -0.01" xyz="0.09 0.01 0.055"/> <!--for jaxon red-->
+    <!-- <origin rpy="-0.01 0.04 -0.01" xyz="0.09 0.01 0.055"/> --> <!--for jaxon red, for jsk leg-->
+    <origin rpy="-0.01 0.0 -0.01" xyz="0.08 0.01 0.055"/> <!--for jaxon red, for kawada leg-->
     <!-- <origin rpy="-0.01 0.01 0.017" xyz="0.10 0.01 0.065"/> --> <!-- For hand -->
   </joint>

Commit message: [hrpsys_ros_bridge_tutorials] Update jaxonred calib param

File: hrpsys_ros_bridge_tutorials/models/JAXON_RED.urdf.xacro (robot description, xacro)
@@ -57,5 +57,5 @@
     <!-- <origin rpy="-0.01 0.04 0.017" xyz="0.095 -0.01 0.055"/> for jaxon -->
     <!-- <origin rpy="-0.01 0.04 -0.01" xyz="0.09 0.01 0.055"/> --> <!--for jaxon red, for jsk leg-->
-    <origin rpy="-0.01 0.0 -0.01" xyz="0.08 0.01 0.055"/> <!--for jaxon red, for kawada leg-->
+    <origin rpy="-0.01 0.04 -0.01" xyz="0.1 0.01 0.07"/>
     <!-- <origin rpy="-0.01 0.01 0.017" xyz="0.10 0.01 0.065"/> --> <!-- For hand -->
   </joint>

Commit message: [hrpsys_ros_bridge_tutorials: update jaxon red calib param

File: hrpsys_ros_bridge_tutorials/models/JAXON_RED.urdf.xacro (robot description, xacro)
@@ -57,5 +57,5 @@
     <!-- <origin rpy="-0.01 0.04 0.017" xyz="0.095 -0.01 0.055"/> for jaxon -->
     <!-- <origin rpy="-0.01 0.04 -0.01" xyz="0.09 0.01 0.055"/> --> <!--for jaxon red, for jsk leg-->
-    <origin rpy="-0.01 0.04 -0.01" xyz="0.1 0.01 0.07"/>
+    <origin rpy="-0.01 0.04 -0.01" xyz="0.1 0.01 0.065"/>
     <!-- <origin rpy="-0.01 0.01 0.017" xyz="0.10 0.01 0.065"/> --> <!-- For hand -->
   </joint>

Commit message: [hrpsys_ros_bridge_tutorials] Update calibration parameter of JAXON_RED

File: hrpsys_ros_bridge_tutorials/models/JAXON_RED.urdf.xacro (robot description, xacro)
@@ -54,9 +54,6 @@
     <parent link="HEAD_LINK1" />
     <child  link="head_root" />
-    <!-- <origin rpy="-0.01 0.01 0.017" xyz="0.08 0.01 0.045"/> --> <!-- For leg -->
-    <!-- <origin rpy="-0.01 0.04 0.017" xyz="0.095 -0.01 0.055"/> for jaxon -->
-    <!-- <origin rpy="-0.01 0.04 -0.01" xyz="0.09 0.01 0.055"/> --> <!--for jaxon red, for jsk leg-->
-    <origin rpy="-0.01 0.04 -0.01" xyz="0.1 0.01 0.065"/>
-    <!-- <origin rpy="-0.01 0.01 0.017" xyz="0.10 0.01 0.065"/> --> <!-- For hand -->
+    <!-- <origin rpy="-0.01 0.04 -0.01" xyz="0.1 0.01 0.65"/> -->
+    <origin rpy="-0.01 0.02 -0.01" xyz="0.1 0.01 0.08"/>
   </joint>
   <!-- HAND -->

Commit message: [JAXON_RED] update camera external parameter

File: hrpsys_ros_bridge_tutorials/models/JAXON_RED.urdf.xacro (robot description, xacro)
@@ -55,5 +55,5 @@
     <child  link="head_root" />
     <!-- <origin rpy="-0.01 0.04 -0.01" xyz="0.1 0.01 0.65"/> -->
-    <origin rpy="-0.01 0.02 -0.01" xyz="0.1 0.01 0.08"/>
+    <origin rpy="-0.025 0.055 0.01" xyz="0.1 -0.015 0.08"/> <!-- 2015.11.24 kakiuchi -->
   </joint>
   <!-- HAND -->

Commit message: add calibration setting for JAXON_RED

File: hrpsys_ros_bridge_tutorials/models/JAXON_RED.urdf.xacro (robot description, xacro)
@@ -57,4 +57,12 @@
     <origin rpy="-0.025 0.055 0.01" xyz="0.1 -0.015 0.08"/> <!-- 2015.11.24 kakiuchi -->
   </joint>
+  <!-- for calibration / original offset of camera_frame
+  <link name="left_camera_optical_frame" />
+  <joint name="left_camera_optical_frame_joint" type="fixed">
+    <parent link="HEAD_LINK1" />
+    <child  link="left_camera_optical_frame" />
+    <origin xyz="0.08 0.035 0.067" rpy="-1.5707960129 0 -1.5707960129"/>
+  </joint>
+  -->
   <!-- HAND -->
   <xacro:include filename="$(find jaxon_description)/urdf/thk_hand003.urdf.xacro" />

Commit message: [JAXON_RED] update jaxon_red camera position

File: hrpsys_ros_bridge_tutorials/models/JAXON_RED.urdf.xacro (robot description, xacro)
@@ -55,5 +55,8 @@
     <child  link="head_root" />
     <!-- <origin rpy="-0.01 0.04 -0.01" xyz="0.1 0.01 0.65"/> -->
-    <origin rpy="-0.025 0.055 0.01" xyz="0.1 -0.015 0.08"/> <!-- 2015.11.24 kakiuchi -->
+    <!-- 2015.11.24 kakiuchi -->
+    <!-- origin rpy="-0.025 0.055 0.01" xyz="0.1 -0.015 0.08"/-->
+    <!-- calibration at 2015.12.09 with jaxon_calibration -->
+    <origin xyz="0.097542410 -0.000296955 0.063307448" rpy="-0.007600616 0.046755703 -0.015569626" />
   </joint>
   <!-- for calibration / original offset of camera_frame

Commit message: [hrpsys_ros_bridge_tutorials] caalibrate mutlisense because JAXON_RED mutlisense mount is modified on 2016/05/30

File: hrpsys_ros_bridge_tutorials/models/JAXON_RED.urdf.xacro (robot description, xacro)
@@ -58,5 +58,7 @@
     <!-- origin rpy="-0.025 0.055 0.01" xyz="0.1 -0.015 0.08"/-->
     <!-- calibration at 2015.12.09 with jaxon_calibration -->
-    <origin xyz="0.097542410 -0.000296955 0.063307448" rpy="-0.007600616 0.046755703 -0.015569626" />
+    <!-- <origin xyz="0.097542410 -0.000296955 0.063307448" rpy="-0.007600616 0.046755703 -0.015569626" /> -->
+    <!-- 2016.6.1 tamura kumagai by modification of mount frame -->
+    <origin rpy="-0.005 0.048 -0.020569626" xyz="0.095 0.003596955 0.075307448"/>
   </joint>
   <!-- for calibration / original offset of camera_frame
