Commit message: fix gazebo files for jaxon simulation

File: hrpsys_gazebo_tutorials/robot_models/JAXON/JAXON_without_multisense.urdf.xacro (robot description, xacro)
@@ -1,11 +1,4 @@
 <robot xmlns:xacro="http://www.ros.org/wiki/xacro" name="JAXON" >
   <xacro:include filename="$(find hrpsys_gazebo_tutorials)/robot_models/JAXON/JAXON.urdf" />
-  <!-- HEAD -->
-  <xacro:include filename="$(find multisense_sl_description)/urdf/multisense_sl_v4.urdf" />
-  <joint name="jaxon_to_multisense" type="fixed">
-    <parent link="HEAD_LINK1" />
-    <child  link="head" />
-    <origin xyz="0.1005 0 0.05625" rpy="0 0 0"/>
-  </joint>
   <!-- HAND -->
   <xacro:include filename="$(find jaxon_description)/urdf/thk_hand003.urdf.xacro" />

Commit message: add multisense urdf of real robot to jaxon_without_multisense xacro

File: hrpsys_gazebo_tutorials/robot_models/JAXON/JAXON_without_multisense.urdf.xacro (robot description, xacro)
@@ -1,4 +1,11 @@
 <robot xmlns:xacro="http://www.ros.org/wiki/xacro" name="JAXON" >
   <xacro:include filename="$(find hrpsys_gazebo_tutorials)/robot_models/JAXON/JAXON.urdf" />
+  <!-- HEAD -->
+  <xacro:include filename="$(find multisense_description)/urdf/multisenseSL.urdf" />
+  <joint name="head_tip_to_multisense" type="fixed">
+    <parent link="HEAD_LINK1" />
+    <child  link="head_root" />
+    <origin rpy="0.004 0.01 0.01" xyz="0.1005 0 0.07625"/>
+  </joint>
   <!-- HAND -->
   <xacro:include filename="$(find jaxon_description)/urdf/thk_hand003.urdf.xacro" />

Commit message: add end-effector joint and links to jaxon xacro. these are added automatically from yaml files in hrpsys_ros_bridge_tutorials, so this change is temporary, and we should use that model.

File: hrpsys_gazebo_tutorials/robot_models/JAXON/JAXON_without_multisense.urdf.xacro (robot description, xacro)
@@ -47,3 +47,64 @@
     </sensor>
   </gazebo>
+  <!-- end-effectors -->
+  <joint name="rfsensor_joint" type="fixed">
+    <origin rpy="3.141593 0.000000 3.141593" xyz="0 0 -0.069"/>
+    <parent link="RLEG_LINK5"/>
+    <child link="rfsensor"/>
+  </joint>
+  <link name="rfsensor"/>
+  <joint name="lfsensor_joint" type="fixed">
+    <origin rpy="3.141593 0.000000 3.141593" xyz="0 0 -0.069"/>
+    <parent link="LLEG_LINK5"/>
+    <child link="lfsensor"/>
+  </joint>
+  <link name="lfsensor"/>
+  <joint name="rhsensor_joint" type="fixed">
+    <origin rpy="-3.141593 -0.000000 2.356196" xyz="0 0 -0.069"/>
+    <parent link="RARM_LINK7"/>
+    <child link="rhsensor"/>
+  </joint>
+  <link name="rhsensor"/>
+  <joint name="lhsensor_joint" type="fixed">
+    <origin rpy="3.141593 -0.000000 -2.356196" xyz="0 0 -0.069"/>
+    <parent link="LARM_LINK7"/>
+    <child link="lhsensor"/>
+  </joint>
+  <link name="lhsensor"/>
+  <joint name="fisheye_joint" type="fixed">
+    <origin rpy="-2.617989 0.000005 -1.570795" xyz="0.147 0 -0.022"/>
+    <parent link="CHEST_LINK2"/>
+    <child link="fisheye"/>
+  </joint>
+  <link name="fisheye"/>
+  <joint name="rleg_end_coords_joint" type="fixed">
+    <origin rpy="0.000000 -0.000000 0.000000" xyz="0 0 -0.1055"/>
+    <parent link="RLEG_LINK5"/>
+    <child link="rleg_end_coords"/>
+  </joint>
+  <link name="rleg_end_coords"/>
+  <joint name="lleg_end_coords_joint" type="fixed">
+    <origin rpy="0.000000 -0.000000 0.000000" xyz="0 0 -0.1055"/>
+    <parent link="LLEG_LINK5"/>
+    <child link="lleg_end_coords"/>
+  </joint>
+  <link name="lleg_end_coords"/>
+  <joint name="rarm_end_coords_joint" type="fixed">
+    <origin rpy="-0.000000 1.570796 0.000000" xyz="0 0 -0.217"/>
+    <parent link="RARM_LINK7"/>
+    <child link="rarm_end_coords"/>
+  </joint>
+  <link name="rarm_end_coords"/>
+  <joint name="larm_end_coords_joint" type="fixed">
+    <origin rpy="-0.000000 1.570796 0.000000" xyz="0 0 -0.217"/>
+    <parent link="LARM_LINK7"/>
+    <child link="larm_end_coords"/>
+  </joint>
+  <link name="larm_end_coords"/>
+  <joint name="head_end_coords_joint" type="fixed">
+    <origin rpy="-0.000000 1.570796 0.000000" xyz="0.1 0.0 0.1"/>
+    <parent link="HEAD_LINK1"/>
+    <child link="head_end_coords"/>
+  </joint>
+  <link name="head_end_coords"/>
 </robot>
