Commit message: fix cube model to use with interactive marker.

File: hrpsys_gazebo_tutorials/environment_models/Cube/Cube.urdf (robot description, URDF)
Before this commit: robot cube-robot, 1 links, 0 joints
Links:
- link nil_link: geometry collision mesh filename=package://hrpsys_gazebo_tutorials/environment_models/Cube/m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 scale=1 1 1; visual mesh filename=package://hrpsys_gazebo_tutorials/environment_models/Cube/m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 scale=1 1 1
